File: pmic-test-board/pmic-test-board.kicad_pcb (KiCad board)
At the start: 4 copper layers, 100 x 100 mm, 200 parts, among them J101 Conn_Coaxial, J102 Conn_Coaxial, J103 Conn_Coaxial, J104 Conn_Coaxial, J105 Conn_01x02_Male, J106 Conn_01x04_Male, J107 Conn_01x04_Male, J108 Conn_02x09_Odd_Even, J109 Conn_Coaxial, J110 Conn_Coaxial, J113 Conn_01x04_Female, J114 Conn_Coaxial, J115 mounting-hole-nc, J116 mounting-hole-nc, J117 mounting-hole-nc, J118 mounting-hole-nc, J202 Conn_01x02_Male, J203 Conn_01x02_Male, J204 Conn_01x02_Male, J205 Conn_01x02_Male, J207 Conn_01x02_Female, J208 Conn_01x04_Female, J301 Conn_Coaxial, J401 Conn_01x02_Male, Q102 BSR202N, Q103 BSR202N, Q104 BSR202N, Q501 BSR202N, Q502 BSR202N, Q503 BSR202N, Q504 BSR202N, SW101 SW_DIP_x08, SW102 SW_Push, SW501 SW_DIP_x08, U101 74LVC2G34, U102 74LVC2G34, U103 W25Q32JVSS, U104 Caravel-QFN, U201 AZ1117-3.3, U202 AZ1117-1.8, U301 AZ431LANTR-G1, U302 DS4424N+, U401 LMH6601, X101 ASE-10.000MHZ-LC-T

Commit message: schematic review and gerber generation
Parts:
- added TP107: TestPoint, wbraun_smd:THM_COMPACT, F.Cu at (118.0, 136.5)
- added TP108: TestPoint, wbraun_smd:THM_COMPACT, F.Cu at (132.8, 138.5)
- added TP109: TestPoint, wbraun_smd:THM_COMPACT, F.Cu at (127.8, 134.5)
- added TP110: TestPoint, wbraun_smd:THM_COMPACT, F.Cu at (155.2, 134.0)
- added TP111: TestPoint, wbraun_smd:THM_COMPACT, F.Cu at (107.5, 138.5)
Connections:
- U401 pad 3: IMON -> /TIA/TIA_VREF
- U401 pad 4: /TIA/TIA_VREF -> IMON
Routing:
- net LOAD_SW: track 34.3 -> 39.8 mm
- net /pmos_val: track 67.4 -> 71.1 mm
- net /timeout_ext: track 85.8 -> 89.3 mm
- net IMON: track 17.0 -> 20.3 mm
- net /TIA/TIA_VREF: track 10.6 -> 13.2 mm, vias 0 -> 2
- net /nmos_val: track 69.0 -> 71.0 mm
- net /TIA/TIA_SENSE: track 19.2 -> 20.5 mm, vias 0 -> 2
