File: pmic-test-board/Load.sch (KiCad schematic (older format))
At the start: 4 parts

Commit message: more schematic capture
Parts:
- Q501: renamed from Q?; footprint (none) -> Package_TO_SOT_SMD:SOT-23
- R501, R502, R503: renamed from R?; footprint (none) -> Resistor_SMD:R_2512_6332Metric
Changed lines of the file:
@@
 $EndDescr
 $Comp
-L Device:R R?
-U 1 1 61AE113C
-P 4450 3200
-F 0 "R?" H 4520 3246 50  0000 L CNN
-F 1 "R" H 4520 3155 50  0000 L CNN
-F 2 "" V 4380 3200 50  0001 C CNN
-F 3 "~" H 4450 3200 50  0001 C CNN
-	1    4450 3200
-	1    0    0    -1
-$EndComp
-$Comp
-L Device:R R?
-U 1 1 61AE182C
-P 4850 3200
-F 0 "R?" H 4920 3246 50  0000 L CNN
-F 1 "R" H 4920 3155 50  0000 L CNN
-F 2 "" V 4780 3200 50  0001 C CNN
-F 3 "~" H 4850 3200 50  0001 C CNN
-	1    4850 3200
-	1    0    0    -1
-$EndComp
-$Comp
-L Device:R R?
-U 1 1 61AE1FEA
-P 5250 3200
-F 0 "R?" H 5320 3246 50  0000 L CNN
-F 1 "R" H 5320 3155 50  0000 L CNN
-F 2 "" V 5180 3200 50  0001 C CNN
-F 3 "~" H 5250 3200 50  0001 C CNN
-	1    5250 3200
-	1    0    0    -1
-$EndComp
-$Comp
-L power:GND #PWR?
+L power:GND #PWR0195
 U 1 1 61AE2759
 P 4450 4100
-F 0 "#PWR?" H 4450 3850 50  0001 C CNN
+F 0 "#PWR0195" H 4450 3850 50  0001 C CNN
 F 1 "GND" H 4455 3927 50  0000 C CNN
 F 2 "" H 4450 4100 50  0001 C CNN
@@
 Wire Wire Line
 	4450 4100 4450 4000
-Text GLabel 4400 2650 0    50   Input ~ 0
-BUCK_VOUT
-Wire Wire Line
-	4400 2650 4450 2650
-Wire Wire Line
-	4450 2650 4450 2900
-Wire Wire Line
-	4450 2900 4850 2900
-Wire Wire Line
-	4850 2900 4850 3050
-Connection ~ 4450 2900
-Wire Wire Line
-	4450 2900 4450 3050
-Wire Wire Line
-	4850 2900 5250 2900
-Wire Wire Line
-	5250 2900 5250 3050
-Connection ~ 4850 2900
-Wire Wire Line
-	4450 3350 4450 3500
-Wire Wire Line
-	4850 3350 4850 3500
-Wire Wire Line
-	4850 3500 4450 3500
-Connection ~ 4450 3500
 Wire Wire Line
 	4450 3500 4450 3600
-Wire Wire Line
-	5250 3350 5250 3500
-Wire Wire Line
-	5250 3500 4850 3500
-Connection ~ 4850 3500
 Text GLabel 4000 3800 0    50   Input ~ 0
 LOAD_SW
@@
 	4000 3800 4150 3800
 $Comp
-L Device:Q_NMOS_GSD Q?
+L Device:Q_NMOS_GSD Q501
 U 1 1 61EA619F
 P 4350 3800
-AR Path="/61AE0010/61EA619F" Ref="Q?"  Part="1"
+AR Path="/61AE0010/61EA619F" Ref="Q501"  Part="1"
 AR Path="/61EA619F" Ref="Q?"  Part="1"
-F 0 "Q?" H 4555 3846 50  0000 L CNN
+F 0 "Q501" H 4555 3846 50  0000 L CNN
 F 1 "BSR202N" H 4555 3755 50  0000 L CNN
-F 2 "" H 4550 3900 50  0001 C CNN
+F 2 "Package_TO_SOT_SMD:SOT-23" H 4550 3900 50  0001 C CNN
 F 3 "~" H 4350 3800 50  0001 C CNN
 F 4 "BSR202NL6327HTSA1" H 4350 3800 50  0001 C CNN "MPN"
@@
 	1    0    0    -1
 $EndComp
+Connection ~ 4850 3500
+Connection ~ 4450 3500
+Wire Wire Line
+	5250 3500 4850 3500
+Wire Wire Line
+	4850 3500 4450 3500
+Wire Wire Line
+	5250 3350 5250 3500
+Wire Wire Line
+	4850 3350 4850 3500
+Wire Wire Line
+	4450 3350 4450 3500
+Connection ~ 4850 2900
+Wire Wire Line
+	5250 2900 5250 3050
+Wire Wire Line
+	4850 2900 5250 2900
+Wire Wire Line
+	4450 2900 4450 3050
+Connection ~ 4450 2900
+Wire Wire Line
+	4850 2900 4850 3050
+Wire Wire Line
+	4450 2900 4850 2900
+Wire Wire Line
+	4450 2650 4450 2900
+Wire Wire Line
+	4400 2650 4450 2650
+Text GLabel 4400 2650 0    50   Input ~ 0
+BUCK_VOUT
+$Comp
+L Device:R R503
+U 1 1 61AE1FEA
+P 5250 3200
+F 0 "R503" H 5320 3246 50  0000 L CNN
+F 1 "R" H 5320 3155 50  0000 L CNN
+F 2 "Resistor_SMD:R_2512_6332Metric" V 5180 3200 50  0001 C CNN
+F 3 "~" H 5250 3200 50  0001 C CNN
+	1    5250 3200
+	1    0    0    -1
+$EndComp
+$Comp
+L Device:R R502
+U 1 1 61AE182C
+P 4850 3200
+F 0 "R502" H 4920 3246 50  0000 L CNN
+F 1 "R" H 4920 3155 50  0000 L CNN
+F 2 "Resistor_SMD:R_2512_6332Metric" V 4780 3200 50  0001 C CNN
+F 3 "~" H 4850 3200 50  0001 C CNN
+	1    4850 3200
+	1    0    0    -1
+$EndComp
+$Comp
+L Device:R R501
+U 1 1 61AE113C
+P 4450 3200
+F 0 "R501" H 4520 3246 50  0000 L CNN
+F 1 "R" H 4520 3155 50  0000 L CNN
+F 2 "Resistor_SMD:R_2512_6332Metric" V 4380 3200 50  0001 C CNN
+F 3 "~" H 4450 3200 50  0001 C CNN
+	1    4450 3200
+	1    0    0    -1
+$EndComp

Commit message: PCB routing done
Parts:
- added Q502, Q503, Q504: BSR202N, Package_TO_SOT_SMD:SOT-23, symbol Device:Q_NMOS_GSD
- added R504, R508, R512, R516: 24, Resistor_SMD:R_2512_6332Metric, symbol Device:R
- added R505, R506, R509, R510, R513, R514: 1k, Resistor_SMD:R_0603_1608Metric, symbol Device:R
- added R507, R511, R515: 10k, Resistor_SMD:R_0603_1608Metric, symbol Device:R
- added SW501: SW_DIP_x08, Button_Switch_THT:SW_DIP_SPSTx08_Slide_6.7x21.88mm_W7.62mm_P2.54mm_LowProfile, symbol Switch:SW_DIP_x08
- R501, R502: value R -> 1k; footprint Resistor_SMD:R_2512_6332Metric -> Resistor_SMD:R_0603_1608Metric
- R503: value R -> 10k; footprint Resistor_SMD:R_2512_6332Metric -> Resistor_SMD:R_0603_1608Metric
Connections:
- net BUCK_VOUT: now also R504.1, R508.1, R512.1, R516.1; no longer R501.1, R502.1, R503.1
- net GND: now also R503.2, Q502.2 (S), Q503.2 (S), Q504.2 (S), R507.2, R511.2, R515.2
- net LOAD_SW: now also SW501.10, SW501.11, SW501.12, SW501.9; no longer Q501.1 (G)
- net at R501.2, R502.2: now also Q501.1 (G), R503.1; no longer Q501.3 (D), R503.2
- new net: Q501.3 (D), R504.2
- new net: Q502.1 (G), R505.2, R506.2, R507.1
- new net: Q502.3 (D), R508.2
- new net: Q503.1 (G), R509.2, R510.2, R511.1
- new net: Q503.3 (D), R512.2
- new net: Q504.1 (G), R513.2, R514.2, R515.1
- new net: Q504.3 (D), R516.2
- new net +3V3: SW501.13, SW501.14, SW501.15, SW501.16
- new net DYN1: R501.1, SW501.8
- new net DYN2: R505.1, SW501.7
- new net DYN3: R509.1, SW501.6
- new net DYN4: R513.1, SW501.5
- new net STAT1: R502.1, SW501.4
- new net STAT2: R506.1, SW501.3
- new net STAT3: R510.1, SW501.2
- new net STAT4: R514.1, SW501.1

Commit message: added test firmware and test results
Parts:
- R501, R502, R505, R506, R509, R510, R513, R514: MPN (none) -> RMCF0603FG1K00
- R503, R507, R511, R515: value 10k -> 4.7k; MPN (none) -> RMCF0603FT4K70
- R504, R508, R512, R516: MPN (none) -> AC2512FK-0724RL
Changed lines of the file:
@@
 P 3750 4050
 F 0 "R503" H 3820 4096 50  0000 L CNN
-F 1 "10k" H 3820 4005 50  0000 L CNN
+F 1 "4.7k" H 3820 4005 50  0000 L CNN
 F 2 "Resistor_SMD:R_0603_1608Metric" V 3680 4050 50  0001 C CNN
 F 3 "~" H 3750 4050 50  0001 C CNN
+F 4 "RMCF0603FT4K70" H 3750 4050 50  0001 C CNN "MPN"
 	1    3750 4050
 	1    0    0    -1
@@
 F 2 "Resistor_SMD:R_0603_1608Metric" V 3680 3450 50  0001 C CNN
 F 3 "~" H 3750 3450 50  0001 C CNN
+F 4 "RMCF0603FG1K00" H 3750 3450 50  0001 C CNN "MPN"
 	1    3750 3450
 	1    0    0    -1
@@
 F 2 "Resistor_SMD:R_0603_1608Metric" V 3280 3450 50  0001 C CNN
 F 3 "~" H 3350 3450 50  0001 C CNN
+F 4 "RMCF0603FG1K00" H 3350 3450 50  0001 C CNN "MPN"
 	1    3350 3450
 	1    0    0    -1
@@
 F 2 "Resistor_SMD:R_2512_6332Metric" V 4380 3250 50  0001 C CNN
 F 3 "~" H 4450 3250 50  0001 C CNN
+F 4 "AC2512FK-0724RL" H 4450 3250 50  0001 C CNN "MPN"
 	1    4450 3250
 	1    0    0    -1
@@
 P 5950 4050
 F 0 "R507" H 6020 4096 50  0000 L CNN
-F 1 "10k" H 6020 4005 50  0000 L CNN
+F 1 "4.7k" H 6020 4005 50  0000 L CNN
 F 2 "Resistor_SMD:R_0603_1608Metric" V 5880 4050 50  0001 C CNN
 F 3 "~" H 5950 4050 50  0001 C CNN
+F 4 "RMCF0603FT4K70" H 5950 4050 50  0001 C CNN "MPN"
 	1    5950 4050
 	1    0    0    -1
@@
 F 2 "Resistor_SMD:R_0603_1608Metric" V 5880 3450 50  0001 C CNN
 F 3 "~" H 5950 3450 50  0001 C CNN
+F 4 "RMCF0603FG1K00" H 5950 3450 50  0001 C CNN "MPN"
 	1    5950 3450
 	1    0    0    -1
@@
 F 2 "Resistor_SMD:R_0603_1608Metric" V 5480 3450 50  0001 C CNN
 F 3 "~" H 5550 3450 50  0001 C CNN
+F 4 "RMCF0603FG1K00" H 5550 3450 50  0001 C CNN "MPN"
 	1    5550 3450
 	1    0    0    -1
@@
 F 2 "Resistor_SMD:R_2512_6332Metric" V 6580 3250 50  0001 C CNN
 F 3 "~" H 6650 3250 50  0001 C CNN
+F 4 "AC2512FK-0724RL" H 6650 3250 50  0001 C CNN "MPN"
 	1    6650 3250
 	1    0    0    -1
@@
 P 8100 3950
 F 0 "R511" H 8170 3996 50  0000 L CNN
-F 1 "10k" H 8170 3905 50  0000 L CNN
+F 1 "4.7k" H 8170 3905 50  0000 L CNN
 F 2 "Resistor_SMD:R_0603_1608Metric" V 8030 3950 50  0001 C CNN
 F 3 "~" H 8100 3950 50  0001 C CNN
+F 4 "RMCF0603FT4K70" H 8100 3950 50  0001 C CNN "MPN"
 	1    8100 3950
 	1    0    0    -1
@@
 F 2 "Resistor_SMD:R_0603_1608Metric" V 8030 3350 50  0001 C CNN
 F 3 "~" H 8100 3350 50  0001 C CNN
+F 4 "RMCF0603FG1K00" H 8100 3350 50  0001 C CNN "MPN"
 	1    8100 3350
 	1    0    0    -1
@@
 F 2 "Resistor_SMD:R_0603_1608Metric" V 7630 3350 50  0001 C CNN
 F 3 "~" H 7700 3350 50  0001 C CNN
+F 4 "RMCF0603FG1K00" H 7700 3350 50  0001 C CNN "MPN"
 	1    7700 3350
 	1    0    0    -1
@@
 F 2 "Resistor_SMD:R_2512_6332Metric" V 8730 3150 50  0001 C CNN
 F 3 "~" H 8800 3150 50  0001 C CNN
+F 4 "AC2512FK-0724RL" H 8800 3150 50  0001 C CNN "MPN"
 	1    8800 3150
 	1    0    0    -1
@@
 P 9950 3950
 F 0 "R515" H 10020 3996 50  0000 L CNN
-F 1 "10k" H 10020 3905 50  0000 L CNN
+F 1 "4.7k" H 10020 3905 50  0000 L CNN
 F 2 "Resistor_SMD:R_0603_1608Metric" V 9880 3950 50  0001 C CNN
 F 3 "~" H 9950 3950 50  0001 C CNN
+F 4 "RMCF0603FT4K70" H 9950 3950 50  0001 C CNN "MPN"
 	1    9950 3950
 	1    0    0    -1
@@
 F 2 "Resistor_SMD:R_0603_1608Metric" V 9880 3350 50  0001 C CNN
 F 3 "~" H 9950 3350 50  0001 C CNN
+F 4 "RMCF0603FG1K00" H 9950 3350 50  0001 C CNN "MPN"
 	1    9950 3350
 	1    0    0    -1
@@
 F 2 "Resistor_SMD:R_0603_1608Metric" V 9480 3350 50  0001 C CNN
 F 3 "~" H 9550 3350 50  0001 C CNN
+F 4 "RMCF0603FG1K00" H 9550 3350 50  0001 C CNN "MPN"
 	1    9550 3350
 	1    0    0    -1
@@
 F 2 "Resistor_SMD:R_2512_6332Metric" V 10580 3150 50  0001 C CNN
 F 3 "~" H 10650 3150 50  0001 C CNN
+F 4 "AC2512FK-0724RL" H 10650 3150 50  0001 C CNN "MPN"
 	1    10650 3150
 	1    0    0    -1
