File: pmic-test-board/Power.sch (KiCad schematic (older format))
At the start: 28 parts

Commit message: more schematic capture
Parts:
- removed C? (x3): 47u, symbol Device:CP1
- removed C?: 470u, symbol Device:CP1
- removed R?: 10m, symbol Device:R
- added C201, C202: 470u, Capacitor_SMD:CP_Elec_10x14.3, symbol Device:CP1
- added C206, C211: 47u, Capacitor_Tantalum_SMD:CP_EIA-3528-12_Kemet-T, symbol Device:CP1
- added R201: 10m, Resistor_SMD:R_Shunt_Ohmite_LVK12, symbol Device:R_Shunt
- C203, C204, C205, C207, C208, C209, C210, C212: renamed from C?; footprint (none) -> Capacitor_SMD:C_0805_2012Metric
- FB201, FB202, FB203: renamed from FB?; footprint (none) -> Inductor_SMD:L_0805_2012Metric
- R202, R203, R204, R205: renamed from R?; footprint (none) -> Resistor_SMD:R_0603_1608Metric
- U201, U202: renamed from U?; footprint (none) -> Package_TO_SOT_SMD:SOT-223-3_TabPin2
- gave numbers to parts that had none: 6
Connections:
- net BUCK_PWR: now also C206.1, R201.1; no longer J202.2 (Pin_2)
- net CTRL_PWR: now also C211.1
- net GND: now also C201.2, C202.2, C206.2, C211.2
- net at C204.1, C205.1, FB201.1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: now also C202.1
- net at C203.1, FB202.1, FB203.2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: now also C201.1, R201.4; no longer J202.1 (Pin_1)
- new net: J202.1 (Pin_1), R201.3
- new net: J202.2 (Pin_2), R201.2

Commit message: PCB routing done
Parts:
- removed C212: 10u, Capacitor_SMD:C_0805_2012Metric, symbol Device:C
- removed J201, J206: Conn_01x02_Male, symbol Connector:Conn_01x02_Male
- removed R205: 0.1, Resistor_SMD:R_0603_1608Metric, symbol Device:R
- added J207: Conn_01x02_Female, wbraun_smd:Terminal-block-plug_2x1_3.5mm-pitch, symbol Connector:Conn_01x02_Female
- added J208: Conn_01x04_Female, wbraun_smd:Terminal-block-plug_4x1_3.5mm-pitch, symbol Connector:Conn_01x04_Female
- added TP201, TP202, TP203: TestPoint, wbraun_smd:THM_COMPACT, symbol Connector:TestPoint
- J202, J203, J204, J205: footprint (none) -> Connector_PinHeader_2.54mm:PinHeader_1x02_P2.54mm_Vertical
- R201: footprint Resistor_SMD:R_Shunt_Ohmite_LVK12 -> wbraun_smd:R_Shunt_Ohmite_LVK12
Connections:
- net +1V8: now also TP202.1
- net BUCK_PWR: now also TP201.1
- net CTRL_PWR: now also TP203.1
- net GND: now also J207.1 (Pin_1), J208.1 (Pin_1), J208.2 (Pin_2)
- net VIN_CTRL: now reaches C202.1, C204.1, C205.1, FB201.1, U201.3 (VI), U202.3 (VI)
- net VIN_PWR: now reaches C201.1, C203.1, FB202.1, FB203.2, R201.4
- net VIN_CONTROL: no longer names the net of FB201.2
- net VIN_CONTROL: now also J207.2 (Pin_2)
- net VIN_POWER: no longer names the net of FB202.2
- net VIN_POWER: now also J208.3 (Pin_3), J208.4 (Pin_4)
Changed lines of the file:
@@
 Connection ~ 5800 1700
 Wire Wire Line
-	6400 1700 6650 1700
+	6400 1700 6500 1700
 Wire Wire Line
 	6650 1700 6650 1750
@@
 Connection ~ 6650 3250
 $Comp
-L power:+3.3VA #PWR0168
-U 1 1 619F0A4D
-P 7800 3250
-F 0 "#PWR0168" H 7800 3100 50  0001 C CNN
-F 1 "+3.3VA" H 7815 3423 50  0000 C CNN
-F 2 "" H 7800 3250 50  0001 C CNN
-F 3 "" H 7800 3250 50  0001 C CNN
-	1    7800 3250
-	1    0    0    -1
-$EndComp
-$Comp
-L Device:R R205
-U 1 1 619F2073
-P 7250 3250
-F 0 "R205" V 7043 3250 50  0000 C CNN
-F 1 "0.1" V 7134 3250 50  0000 C CNN
-F 2 "Resistor_SMD:R_0603_1608Metric" V 7180 3250 50  0001 C CNN
-F 3 "~" H 7250 3250 50  0001 C CNN
-	1    7250 3250
-	0    1    1    0
-$EndComp
-$Comp
-L Device:C C212
-U 1 1 619F26C8
-P 7800 3500
-F 0 "C212" H 7915 3546 50  0000 L CNN
-F 1 "10u" H 7915 3455 50  0000 L CNN
-F 2 "Capacitor_SMD:C_0805_2012Metric" H 7838 3350 50  0001 C CNN
-F 3 "~" H 7800 3500 50  0001 C CNN
-	1    7800 3500
-	1    0    0    -1
-$EndComp
-Wire Wire Line
-	7100 3250 7000 3250
-Wire Wire Line
-	7000 3250 7000 2900
-Wire Wire Line
-	5750 2900 5750 3250
-$Comp
-L power:GND #PWR0169
-U 1 1 619F5DAE
-P 7800 3800
-F 0 "#PWR0169" H 7800 3550 50  0001 C CNN
-F 1 "GND" H 7805 3627 50  0000 C CNN
-F 2 "" H 7800 3800 50  0001 C CNN
-F 3 "" H 7800 3800 50  0001 C CNN
-	1    7800 3800
-	1    0    0    -1
-$EndComp
-Wire Wire Line
-	7800 3650 7800 3800
-Wire Wire Line
-	7800 3350 7800 3250
-Connection ~ 7800 3250
-Wire Wire Line
-	1900 1700 2450 1700
-Text GLabel 1900 1700 0    50   Input ~ 0
-VIN_CONTROL
-$Comp
-L Connector:Conn_01x02_Male J206
-U 1 1 619F9A41
-P 7200 3650
-F 0 "J206" V 7000 3600 50  0000 L CNN
-F 1 "Conn_01x02_Male" V 7100 3350 50  0000 L CNN
-F 2 "" H 7200 3650 50  0001 C CNN
-F 3 "~" H 7200 3650 50  0001 C CNN
-	1    7200 3650
-	0    -1   -1   0
-$EndComp
-$Comp
 L Connector:Conn_01x02_Male J204
 U 1 1 619FBD4B
@@
 F 0 "J204" V 6000 3600 50  0000 L CNN
 F 1 "Conn_01x02_Male" V 6100 3350 50  0000 L CNN
-F 2 "" H 6200 3650 50  0001 C CNN
+F 2 "Connector_PinHeader_2.54mm:PinHeader_1x02_P2.54mm_Vertical" H 6200 3650 50  0001 C CNN
 F 3 "~" H 6200 3650 50  0001 C CNN
 	1    6200 3650
@@
 F 0 "J203" V 6000 2050 50  0000 L CNN
 F 1 "Conn_01x02_Male" V 6100 1800 50  0000 L CNN
-F 2 "" H 6200 2100 50  0001 C CNN
+F 2 "Connector_PinHeader_2.54mm:PinHeader_1x02_P2.54mm_Vertical" H 6200 2100 50  0001 C CNN
 F 3 "~" H 6200 2100 50  0001 C CNN
 	1    6200 2100
@@
 	6100 3450 6100 3250
 Connection ~ 6100 3250
-Wire Wire Line
-	7200 3450 7100 3450
-Wire Wire Line
-	7100 3450 7100 3250
-Connection ~ 7100 3250
-Wire Wire Line
-	7300 3450 7400 3450
-Wire Wire Line
-	7400 3450 7400 3250
-Wire Wire Line
-	7400 3250 7800 3250
-Connection ~ 7400 3250
-Wire Wire Line
-	7000 2900 5750 2900
-Text GLabel 2650 5400 0    50   Input ~ 0
-VIN_POWER
 $Comp
 L Device:C C203
@@
 	1    0    0    -1
 $EndComp
-Wire Wire Line
-	2650 5400 3050 5400
 Wire Wire Line
 	3250 5400 3400 5400
@@
 F 0 "J202" V 4150 5750 50  0000 L CNN
 F 1 "Conn_01x02_Male" V 4250 5500 50  0000 L CNN
-F 2 "" H 4350 5800 50  0001 C CNN
+F 2 "Connector_PinHeader_2.54mm:PinHeader_1x02_P2.54mm_Vertical" H 4350 5800 50  0001 C CNN
 F 3 "~" H 4350 5800 50  0001 C CNN
 	1    4350 5800
@@
 F 0 "J205" V 6100 5700 50  0000 L CNN
 F 1 "Conn_01x02_Male" V 6200 5450 50  0000 L CNN
-F 2 "" H 6300 5750 50  0001 C CNN
+F 2 "Connector_PinHeader_2.54mm:PinHeader_1x02_P2.54mm_Vertical" H 6300 5750 50  0001 C CNN
 F 3 "~" H 6300 5750 50  0001 C CNN
 	1    6300 5750
@@
 $EndComp
 Wire Wire Line
-	6500 5350 6750 5350
+	6500 5350 6650 5350
 Wire Wire Line
 	6750 5350 6750 5500
@@
 Text GLabel 4800 5400 2    50   Input ~ 0
 BUCK_PWR
-$Comp
-L Connector:Conn_01x02_Male J201
-U 1 1 61A600E3
-P 3750 4750
-F 0 "J201" V 3550 4700 50  0000 L CNN
-F 1 "Conn_01x02_Male" V 3650 4450 50  0000 L CNN
-F 2 "" H 3750 4750 50  0001 C CNN
-F 3 "~" H 3750 4750 50  0001 C CNN
-	1    3750 4750
-	0    1    1    0
-$EndComp
-$Comp
-L power:GND #PWR0172
-U 1 1 61A61C00
-P 3650 5050
-F 0 "#PWR0172" H 3650 4800 50  0001 C CNN
-F 1 "GND" H 3655 4877 50  0000 C CNN
-F 2 "" H 3650 5050 50  0001 C CNN
-F 3 "" H 3650 5050 50  0001 C CNN
-	1    3650 5050
-	1    0    0    -1
-$EndComp
 Wire Wire Line
 	3750 4950 3750 5050
@@
 	3750 5050 3950 5050
 Connection ~ 3950 5050
-Wire Wire Line
-	3650 4950 3650 5050
 Text GLabel 6750 5350 2    50   Input ~ 0
 CTRL_PWR
@@
 F 0 "R201" V 4175 5400 50  0000 C CNN
 F 1 "10m" V 4266 5400 50  0000 C CNN
-F 2 "Resistor_SMD:R_Shunt_Ohmite_LVK12" V 4330 5400 50  0001 C CNN
+F 2 "wbraun_smd:R_Shunt_Ohmite_LVK12" V 4330 5400 50  0001 C CNN
 F 3 "~" H 4400 5400 50  0001 C CNN
 F 4 "LVK12R010CER" V 4400 5400 50  0001 C CNN "MPN"
@@
 	3950 5400 4200 5400
 Wire Wire Line
-	4600 5400 4800 5400
+	4600 5400 4700 5400
 Wire Wire Line
 	4500 5600 4500 5550
 Wire Wire Line
 	4300 5600 4300 5550
+$Comp
+L Connector:Conn_01x02_Female J?
+U 1 1 6218656E
+P 1550 1800
+AR Path="/6218656E" Ref="J?"  Part="1"
+AR Path="/6198672D/6218656E" Ref="J207"  Part="1"
+F 0 "J207" H 1442 1475 50  0000 C CNN
+F 1 "Conn_01x02_Female" H 1442 1566 50  0000 C CNN
+F 2 "wbraun_smd:Terminal-block-plug_2x1_3.5mm-pitch" H 1550 1800 50  0001 C CNN
+F 3 "~" H 1550 1800 50  0001 C CNN
+	1    1550 1800
+	-1   0    0    1
+$EndComp
+Wire Wire Line
+	1750 1700 2450 1700
+$Comp
+L power:GND #PWR0235
+U 1 1 6218AF6E
+P 1850 1850
+F 0 "#PWR0235" H 1850 1600 50  0001 C CNN
+F 1 "GND" H 1855 1677 50  0000 C CNN
+F 2 "" H 1850 1850 50  0001 C CNN
+F 3 "" H 1850 1850 50  0001 C CNN
+	1    1850 1850
+	1    0    0    -1
+$EndComp
+Wire Wire Line
+	1750 1800 1850 1800
+Wire Wire Line
+	1850 1800 1850 1850
+Text Label 3200 1700 0    50   ~ 0
+VIN_CTRL
+Text Label 3950 5050 0    50   ~ 0
+VIN_PWR
+$Comp
+L Connector:Conn_01x04_Female J208
+U 1 1 6218F6B5
+P 1750 5600
+F 0 "J208" H 1642 5885 50  0000 C CNN
+F 1 "Conn_01x04_Female" H 1642 5794 50  0000 C CNN
+F 2 "wbraun_smd:Terminal-block-plug_4x1_3.5mm-pitch" H 1750 5600 50  0001 C CNN
+F 3 "~" H 1750 5600 50  0001 C CNN
+F 4 "0395021004" H 1750 5600 50  0001 C CNN "MPN"
+	1    1750 5600
+	-1   0    0    1
+$EndComp
+Wire Wire Line
+	1950 5400 2150 5400
+Wire Wire Line
+	1950 5500 2150 5500
+Wire Wire Line
+	2150 5500 2150 5400
+Connection ~ 2150 5400
+Wire Wire Line
+	2150 5400 3050 5400
+$Comp
+L power:GND #PWR0236
+U 1 1 62194784
+P 2150 5750
+F 0 "#PWR0236" H 2150 5500 50  0001 C CNN
+F 1 "GND" H 2155 5577 50  0000 C CNN
+F 2 "" H 2150 5750 50  0001 C CNN
+F 3 "" H 2150 5750 50  0001 C CNN
+	1    2150 5750
+	1    0    0    -1
+$EndComp
+Wire Wire Line
+	1950 5600 2150 5600
+Wire Wire Line
+	2150 5600 2150 5700
+Wire Wire Line
+	1950 5700 2150 5700
+Connection ~ 2150 5700
+Wire Wire Line
+	2150 5700 2150 5750
+$Comp
+L Connector:TestPoint TP202
+U 1 1 6244670A
+P 6500 1350
+F 0 "TP202" H 6558 1468 50  0000 L CNN
+F 1 "TestPoint" H 6558 1377 50  0000 L CNN
+F 2 "wbraun_smd:THM_COMPACT" H 6700 1350 50  0001 C CNN
+F 3 "~" H 6700 1350 50  0001 C CNN
+	1    6500 1350
+	1    0    0    -1
+$EndComp
+$Comp
+L Connector:TestPoint TP203
+U 1 1 62447E34
+P 6650 5150
+F 0 "TP203" H 6708 5268 50  0000 L CNN
+F 1 "TestPoint" H 6708 5177 50  0000 L CNN
+F 2 "wbraun_smd:THM_COMPACT" H 6850 5150 50  0001 C CNN
+F 3 "~" H 6850 5150 50  0001 C CNN
+	1    6650 5150
+	1    0    0    -1
+$EndComp
+$Comp
+L Connector:TestPoint TP201
+U 1 1 62449469
+P 4700 5300
+F 0 "TP201" H 4758 5418 50  0000 L CNN
+F 1 "TestPoint" H 4758 5327 50  0000 L CNN
+F 2 "wbraun_smd:THM_COMPACT" H 4900 5300 50  0001 C CNN
+F 3 "~" H 4900 5300 50  0001 C CNN
+	1    4700 5300
+	1    0    0    -1
+$EndComp
+Wire Wire Line
+	4700 5300 4700 5400
+Connection ~ 4700 5400
+Wire Wire Line
+	4700 5400 4800 5400
+Wire Wire Line
+	6650 5150 6650 5350
+Connection ~ 6650 5350
+Wire Wire Line
+	6650 5350 6750 5350
+Wire Wire Line
+	6500 1350 6500 1700
+Connection ~ 6500 1700
+Wire Wire Line
+	6500 1700 6650 1700
 $EndSCHEMATC

Commit message: added test firmware and test results
Parts:
- C203, C204, C205, C207, C208, C209, C210: MPN (none) -> CL21B106KPQNFNE
- C206, C211: MPN T520B476M008ATE035 -> T520B476M010ATE035
- FB201, FB202, FB203: MPN (none) -> 742792012
- J207: MPN (none) -> 1844210
- R202, R203, R204: MPN (none) -> ERJ-3BSFR10V
- TP201, TP202, TP203: MPN (none) -> 5119
- U201: MPN (none) -> AZ1117IH-3.3TRG1
- U202: MPN (none) -> AZ1117CH-1.8TRG1
Changed lines of the file:
@@
 F 2 "Package_TO_SOT_SMD:SOT-223-3_TabPin2" H 5150 1950 50  0001 C CIN
 F 3 "https://www.diodes.com/assets/Datasheets/AZ1117.pdf" H 5150 1700 50  0001 C CNN
+F 4 "AZ1117CH-1.8TRG1" H 5150 1700 50  0001 C CNN "MPN"
 	1    5150 1700
 	1    0    0    -1
@@
 F 2 "Package_TO_SOT_SMD:SOT-223-3_TabPin2" H 5100 3500 50  0001 C CIN
 F 3 "https://www.diodes.com/assets/Datasheets/AZ1117.pdf" H 5100 3250 50  0001 C CNN
+F 4 "AZ1117IH-3.3TRG1" H 5100 3250 50  0001 C CNN "MPN"
 	1    5100 3250
 	1    0    0    -1
@@
 F 2 "Capacitor_SMD:C_0805_2012Metric" H 4488 1750 50  0001 C CNN
 F 3 "~" H 4450 1900 50  0001 C CNN
+F 4 "CL21B106KPQNFNE" H 4450 1900 50  0001 C CNN "MPN"
 	1    4450 1900
 	1    0    0    -1
@@
 F 2 "Capacitor_SMD:C_0805_2012Metric" H 4538 3300 50  0001 C CNN
 F 3 "~" H 4500 3450 50  0001 C CNN
+F 4 "CL21B106KPQNFNE" H 4500 3450 50  0001 C CNN "MPN"
 	1    4500 3450
 	1    0    0    -1
@@
 F 2 "Capacitor_SMD:C_0805_2012Metric" H 5838 1750 50  0001 C CNN
 F 3 "~" H 5800 1900 50  0001 C CNN
+F 4 "CL21B106KPQNFNE" H 5800 1900 50  0001 C CNN "MPN"
 	1    5800 1900
 	1    0    0    -1
@@
 F 2 "Capacitor_SMD:C_0805_2012Metric" H 5788 3350 50  0001 C CNN
 F 3 "~" H 5750 3500 50  0001 C CNN
+F 4 "CL21B106KPQNFNE" H 5750 3500 50  0001 C CNN "MPN"
 	1    5750 3500
 	1    0    0    -1
@@
 F 2 "Resistor_SMD:R_0603_1608Metric" V 6180 1700 50  0001 C CNN
 F 3 "~" H 6250 1700 50  0001 C CNN
+F 4 "ERJ-3BSFR10V" H 6250 1700 50  0001 C CNN "MPN"
 	1    6250 1700
 	0    1    1    0
@@
 F 2 "Resistor_SMD:R_0603_1608Metric" V 6180 3250 50  0001 C CNN
 F 3 "~" H 6250 3250 50  0001 C CNN
+F 4 "ERJ-3BSFR10V" H 6250 3250 50  0001 C CNN "MPN"
 	1    6250 3250
 	0    1    1    0
@@
 F 2 "Capacitor_SMD:C_0805_2012Metric" H 6688 3350 50  0001 C CNN
 F 3 "~" H 6650 3500 50  0001 C CNN
+F 4 "CL21B106KPQNFNE" H 6650 3500 50  0001 C CNN "MPN"
 	1    6650 3500
 	1    0    0    -1
@@
 F 2 "Capacitor_SMD:C_0805_2012Metric" H 6688 1750 50  0001 C CNN
 F 3 "~" H 6650 1900 50  0001 C CNN
+F 4 "CL21B106KPQNFNE" H 6650 1900 50  0001 C CNN "MPN"
 	1    6650 1900
 	1    0    0    -1
@@
 F 2 "Inductor_SMD:L_0805_2012Metric" V 3080 5400 50  0001 C CNN
 F 3 "~" H 3150 5400 50  0001 C CNN
+F 4 "742792012" H 3150 5400 50  0001 C CNN "MPN"
 	1    3150 5400
 	0    1    1    0
@@
 F 2 "Inductor_SMD:L_0805_2012Metric" V 2480 1700 50  0001 C CNN
 F 3 "~" H 2550 1700 50  0001 C CNN
+F 4 "742792012" H 2550 1700 50  0001 C CNN "MPN"
 	1    2550 1700
 	0    1    1    0
@@
 F 2 "Capacitor_SMD:C_0805_2012Metric" H 3988 5550 50  0001 C CNN
 F 3 "~" H 3950 5700 50  0001 C CNN
+F 4 "CL21B106KPQNFNE" H 3950 5700 50  0001 C CNN "MPN"
 	1    3950 5700
 	1    0    0    -1
@@
 F 2 "Inductor_SMD:L_0805_2012Metric" V 5830 5350 50  0001 C CNN
 F 3 "~" H 5900 5350 50  0001 C CNN
+F 4 "742792012" H 5900 5350 50  0001 C CNN "MPN"
 	1    5900 5350
 	0    1    1    0
@@
 F 2 "Resistor_SMD:R_0603_1608Metric" V 6280 5350 50  0001 C CNN
 F 3 "~" H 6350 5350 50  0001 C CNN
+F 4 "ERJ-3BSFR10V" H 6350 5350 50  0001 C CNN "MPN"
 	1    6350 5350
 	0    1    1    0
@@
 F 2 "Capacitor_Tantalum_SMD:CP_EIA-3528-12_Kemet-T" H 4800 5700 50  0001 C CNN
 F 3 "~" H 4800 5700 50  0001 C CNN
-F 4 "T520B476M008ATE035" H 4800 5700 50  0001 C CNN "MPN"
+F 4 "T520B476M010ATE035" H 4800 5700 50  0001 C CNN "MPN"
 	1    4800 5700
 	1    0    0    -1
@@
 F 2 "Capacitor_Tantalum_SMD:CP_EIA-3528-12_Kemet-T" H 6750 5650 50  0001 C CNN
 F 3 "~" H 6750 5650 50  0001 C CNN
-F 4 "T520B476M008ATE035" H 6750 5650 50  0001 C CNN "MPN"
+F 4 "T520B476M010ATE035" H 6750 5650 50  0001 C CNN "MPN"
 	1    6750 5650
 	1    0    0    -1
@@
 F 2 "wbraun_smd:Terminal-block-plug_2x1_3.5mm-pitch" H 1550 1800 50  0001 C CNN
 F 3 "~" H 1550 1800 50  0001 C CNN
+F 4 "1844210" H 1550 1800 50  0001 C CNN "MPN"
 	1    1550 1800
 	-1   0    0    1
@@
 F 2 "wbraun_smd:THM_COMPACT" H 6700 1350 50  0001 C CNN
 F 3 "~" H 6700 1350 50  0001 C CNN
+F 4 "5119" H 6500 1350 50  0001 C CNN "MPN"
 	1    6500 1350
 	1    0    0    -1
@@
 F 2 "wbraun_smd:THM_COMPACT" H 6850 5150 50  0001 C CNN
 F 3 "~" H 6850 5150 50  0001 C CNN
+F 4 "5119" H 6650 5150 50  0001 C CNN "MPN"
 	1    6650 5150
 	1    0    0    -1
@@
 F 2 "wbraun_smd:THM_COMPACT" H 4900 5300 50  0001 C CNN
 F 3 "~" H 4900 5300 50  0001 C CNN
+F 4 "5119" H 4700 5300 50  0001 C CNN "MPN"
 	1    4700 5300
 	1    0    0    -1
